File: kicad/pcb-project/pcb-project.kicad_sch (KiCad schematic)
At the start: 13 parts, among them J1 GND, J2 VCC, J3 LOGIC CONN, U1 74HC237

Commit message: Convert schematic to board design
Parts:
- D1, D5: value 2V RED -> 2V; footprint (none) -> Connector_PinSocket_2.54mm:PinSocket_1x02_P2.54mm_Vertical
- D2, D6: value 2V YLW -> 2V; footprint (none) -> Connector_PinSocket_2.54mm:PinSocket_1x02_P2.54mm_Vertical
- D3, D7: value 2V GRN -> 2V; footprint (none) -> Connector_PinSocket_2.54mm:PinSocket_1x02_P2.54mm_Vertical
- D4, D8: value 3V BLU -> 3V; footprint (none) -> Connector_PinSocket_2.54mm:PinSocket_1x02_P2.54mm_Vertical
- J1, J2: footprint (none) -> Connector_PinSocket_2.54mm:PinSocket_1x08_P2.54mm_Vertical
- J3: footprint (none) -> Connector_PinSocket_2.54mm:PinSocket_1x06_P2.54mm_Vertical
- R1: footprint (none) -> Resistor_THT:R_Axial_DIN0204_L3.6mm_D1.6mm_P1.90mm_Vertical
- U1: footprint (none) -> footprints:NS16
Changed lines of the file:
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@@
       (effects (font (size 1.27 1.27)) (justify left))
     )
-    (property "Footprint" "" (id 2) (at 183.642 43.18 90)
+    (property "Footprint" "Resistor_THT:R_Axial_DIN0204_L3.6mm_D1.6mm_P1.90mm_Vertical" (id 2) (at 183.642 43.18 90)
       (effects (font (size 1.27 1.27)) hide)
     )
@@
     (in_bom yes) (on_board yes)
     (property "Reference" "D8" (id 0) (at 181.61 76.2 0))
-    (property "Value" "3V BLU" (id 1) (at 181.61 78.74 0))
-    (property "Footprint" "" (id 2) (at 181.61 72.39 0)
+    (property "Value" "3V" (id 1) (at 181.61 78.74 0))
+    (property "Footprint" "Connector_PinSocket_2.54mm:PinSocket_1x02_P2.54mm_Vertical" (id 2) (at 181.61 72.39 0)
       (effects (font (size 1.27 1.27)) hide)
     )
@@
     (property "Reference" "J1" (id 0) (at 109.22 27.94 90))
     (property "Value" "GND" (id 1) (at 109.22 30.48 90))
-    (property "Footprint" "" (id 2) (at 107.95 34.29 0)
+    (property "Footprint" "Connector_PinSocket_2.54mm:PinSocket_1x08_P2.54mm_Vertical" (id 2) (at 107.95 34.29 0)
       (effects (font (size 1.27 1.27)) hide)
     )
@@
     (property "Reference" "J3" (id 0) (at 111.76 63.5 0))
     (property "Value" "LOGIC CONN" (id 1) (at 111.76 66.04 0))
-    (property "Footprint" "" (id 2) (at 121.92 67.31 0)
+    (property "Footprint" "Connector_PinSocket_2.54mm:PinSocket_1x06_P2.54mm_Vertical" (id 2) (at 121.92 67.31 0)
       (effects (font (size 1.27 1.27)) hide)
     )
@@
     (in_bom yes) (on_board yes)
     (property "Reference" "D5" (id 0) (at 158.75 76.2 0))
-    (property "Value" "2V RED" (id 1) (at 158.75 78.74 0))
-    (property "Footprint" "" (id 2) (at 158.75 64.77 0)
+    (property "Value" "2V" (id 1) (at 158.75 78.74 0))
+    (property "Footprint" "Connector_PinSocket_2.54mm:PinSocket_1x02_P2.54mm_Vertical" (id 2) (at 158.75 64.77 0)
       (effects (font (size 1.27 1.27)) hide)
     )
@@
       (effects (font (size 1.27 1.27)) (justify left))
     )
-    (property "Footprint" "" (id 2) (at 142.24 64.77 0)
+    (property "Footprint" "footprints:NS16" (id 2) (at 142.24 64.77 0)
       (effects (font (size 1.27 1.27)) hide)
     )
@@
     (in_bom yes) (on_board yes)
     (property "Reference" "D2" (id 0) (at 166.37 46.99 0))
-    (property "Value" "2V YLW" (id 1) (at 166.37 49.53 0))
-    (property "Footprint" "" (id 2) (at 166.37 57.15 0)
+    (property "Value" "2V" (id 1) (at 166.37 49.53 0))
+    (property "Footprint" "Connector_PinSocket_2.54mm:PinSocket_1x02_P2.54mm_Vertical" (id 2) (at 166.37 57.15 0)
       (effects (font (size 1.27 1.27)) hide)
     )
@@
     (in_bom yes) (on_board yes)
     (property "Reference" "D3" (id 0) (at 173.99 46.99 0))
-    (property "Value" "2V GRN" (id 1) (at 173.99 49.53 0))
-    (property "Footprint" "" (id 2) (at 173.99 59.69 0)
+    (property "Value" "2V" (id 1) (at 173.99 49.53 0))
+    (property "Footprint" "Connector_PinSocket_2.54mm:PinSocket_1x02_P2.54mm_Vertical" (id 2) (at 173.99 59.69 0)
       (effects (font (size 1.27 1.27)) hide)
     )
@@
     (in_bom yes) (on_board yes)
     (property "Reference" "D7" (id 0) (at 173.99 76.2 0))
-    (property "Value" "2V GRN" (id 1) (at 173.99 78.74 0))
-    (property "Footprint" "" (id 2) (at 173.99 69.85 0)
+    (property "Value" "2V" (id 1) (at 173.99 78.74 0))
+    (property "Footprint" "Connector_PinSocket_2.54mm:PinSocket_1x02_P2.54mm_Vertical" (id 2) (at 173.99 69.85 0)
       (effects (font (size 1.27 1.27)) hide)
     )
@@
     (in_bom yes) (on_board yes)
     (property "Reference" "D4" (id 0) (at 181.61 46.99 0))
-    (property "Value" "3V BLU" (id 1) (at 181.61 49.53 0))
-    (property "Footprint" "" (id 2) (at 181.61 62.23 0)
+    (property "Value" "3V" (id 1) (at 181.61 49.53 0))
+    (property "Footprint" "Connector_PinSocket_2.54mm:PinSocket_1x02_P2.54mm_Vertical" (id 2) (at 181.61 62.23 0)
       (effects (font (size 1.27 1.27)) hide)
     )
@@
     (in_bom yes) (on_board yes)
     (property "Reference" "D1" (id 0) (at 158.75 46.99 0))
-    (property "Value" "2V RED" (id 1) (at 158.75 49.53 0))
-    (property "Footprint" "" (id 2) (at 158.75 54.61 0)
+    (property "Value" "2V" (id 1) (at 158.75 49.53 0))
+    (property "Footprint" "Connector_PinSocket_2.54mm:PinSocket_1x02_P2.54mm_Vertical" (id 2) (at 158.75 54.61 0)
       (effects (font (size 1.27 1.27)) hide)
     )
@@
     (in_bom yes) (on_board yes)
     (property "Reference" "J2" (id 0) (at 109.22 52.07 90))
-    (property "Value" "VCC" (id 1) (at 116.84 52.07 90))
-    (property "Footprint" "" (id 2) (at 110.49 48.26 0)
+    (property "Value" "VCC" (id 1) (at 109.22 54.61 90))
+    (property "Footprint" "Connector_PinSocket_2.54mm:PinSocket_1x08_P2.54mm_Vertical" (id 2) (at 110.49 48.26 0)
       (effects (font (size 1.27 1.27)) hide)
     )
@@
     (in_bom yes) (on_board yes)
     (property "Reference" "D6" (id 0) (at 166.37 76.2 0))
-    (property "Value" "2V YLW" (id 1) (at 166.37 78.74 0))
-    (property "Footprint" "" (id 2) (at 166.37 67.31 0)
+    (property "Value" "2V" (id 1) (at 166.37 78.74 0))
+    (property "Footprint" "Connector_PinSocket_2.54mm:PinSocket_1x02_P2.54mm_Vertical" (id 2) (at 166.37 67.31 0)
       (effects (font (size 1.27 1.27)) hide)
     )
@@
     )
     (path "/c39b5135-fbe0-4931-ad80-ed9c1070d5dd"
-      (reference "D1") (unit 1) (value "2V RED") (footprint "")
+      (reference "D1") (unit 1) (value "2V") (footprint "Connector_PinSocket_2.54mm:PinSocket_1x02_P2.54mm_Vertical")
     )
     (path "/80ca8f03-ac03-4ce8-97d6-b7a0b58fe516"
-      (reference "D2") (unit 1) (value "2V YLW") (footprint "")
+      (reference "D2") (unit 1) (value "2V") (footprint "Connector_PinSocket_2.54mm:PinSocket_1x02_P2.54mm_Vertical")
     )
     (path "/ad021c76-b6ad-49d9-88b7-069b692b6254"
-      (reference "D3") (unit 1) (value "2V GRN") (footprint "")
+      (reference "D3") (unit 1) (value "2V") (footprint "Connector_PinSocket_2.54mm:PinSocket_1x02_P2.54mm_Vertical")
     )
     (path "/bdafbc26-1efa-49e3-b445-a7ce4c7644bc"
-      (reference "D4") (unit 1) (value "3V BLU") (footprint "")
+      (reference "D4") (unit 1) (value "3V") (footprint "Connector_PinSocket_2.54mm:PinSocket_1x02_P2.54mm_Vertical")
     )
     (path "/64e62240-1896-4ac4-9bd9-c6d04c7ea6c6"
-      (reference "D5") (unit 1) (value "2V RED") (footprint "")
+      (reference "D5") (unit 1) (value "2V") (footprint "Connector_PinSocket_2.54mm:PinSocket_1x02_P2.54mm_Vertical")
     )
     (path "/f5e42cc6-743f-4bdd-8ca5-932d4c52bcd5"
-      (reference "D6") (unit 1) (value "2V YLW") (footprint "")
+      (reference "D6") (unit 1) (value "2V") (footprint "Connector_PinSocket_2.54mm:PinSocket_1x02_P2.54mm_Vertical")
     )
     (path "/b65e7d9d-211f-494c-97b8-0375b796e84e"
-      (reference "D7") (unit 1) (value "2V GRN") (footprint "")
+      (reference "D7") (unit 1) (value "2V") (footprint "Connector_PinSocket_2.54mm:PinSocket_1x02_P2.54mm_Vertical")
     )
     (path "/22f44d6a-6c10-4739-9703-7e48601c639c"
-      (reference "D8") (unit 1) (value "3V BLU") (footprint "")
+      (reference "D8") (unit 1) (value "3V") (footprint "Connector_PinSocket_2.54mm:PinSocket_1x02_P2.54mm_Vertical")
     )
     (path "/3d92ab62-134a-4ba8-bb93-98169739d76f"
-      (reference "J1") (unit 1) (value "GND") (footprint "")
+      (reference "J1") (unit 1) (value "GND") (footprint "Connector_PinSocket_2.54mm:PinSocket_1x08_P2.54mm_Vertical")
     )
     (path "/c4906877-f34e-41ea-9593-c886178643dc"
-      (reference "J2") (unit 1) (value "VCC") (footprint "")
+      (reference "J2") (unit 1) (value "VCC") (footprint "Connector_PinSocket_2.54mm:PinSocket_1x08_P2.54mm_Vertical")
     )
     (path "/5a5b773e-8175-42a8-b6b9-e317caca901e"
-      (reference "J3") (unit 1) (value "LOGIC CONN") (footprint "")
+      (reference "J3") (unit 1) (value "LOGIC CONN") (footprint "Connector_PinSocket_2.54mm:PinSocket_1x06_P2.54mm_Vertical")
     )
     (path "/0661d9e7-9725-45e0-99b3-6e9764bee718"
-      (reference "R1") (unit 1) (value "330") (footprint "")
+      (reference "R1") (unit 1) (value "330") (footprint "Resistor_THT:R_Axial_DIN0204_L3.6mm_D1.6mm_P1.90mm_Vertical")
     )
     (path "/6eb8a12c-f7dd-45db-ac57-5cf35b00d623"
-      (reference "U1") (unit 1) (value "74HC237") (footprint "")
-    )
-  )
+      (reference "U1") (unit 1) (value "74HC237") (footprint "footprints:NS16")
+    )
+  )

Commit message: Make annotations and wiring more readable
Parts:
- renumbered J1 to GND1, J3 to J1, J2 to VCC1
Changed lines of the file:
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@@
   (symbol (lib_id "Connector_Generic:Conn_01x08") (at 107.95 34.29 90) (unit 1)
     (in_bom yes) (on_board yes) (fields_autoplaced)
-    (property "Reference" "J1" (id 0) (at 109.22 27.94 90))
+    (property "Reference" "GND1" (id 0) (at 109.22 27.94 90))
     (property "Value" "GND" (id 1) (at 109.22 30.48 90))
     (property "Footprint" "Connector_PinSocket_2.54mm:PinSocket_1x08_P2.54mm_Vertical" (id 2) (at 107.95 34.29 0)
@@
   (symbol (lib_id "Connector_Generic:Conn_01x06") (at 121.92 67.31 180) (unit 1)
     (in_bom yes) (on_board yes)
-    (property "Reference" "J3" (id 0) (at 111.76 63.5 0))
+    (property "Reference" "J1" (id 0) (at 111.76 63.5 0))
     (property "Value" "LOGIC CONN" (id 1) (at 111.76 66.04 0))
     (property "Footprint" "Connector_PinSocket_2.54mm:PinSocket_1x06_P2.54mm_Vertical" (id 2) (at 121.92 67.31 0)
@@
   (symbol (lib_id "Connector_Generic:Conn_01x08") (at 110.49 48.26 270) (unit 1)
     (in_bom yes) (on_board yes)
-    (property "Reference" "J2" (id 0) (at 109.22 52.07 90))
+    (property "Reference" "VCC1" (id 0) (at 109.22 52.07 90))
     (property "Value" "VCC" (id 1) (at 109.22 54.61 90))
     (property "Footprint" "Connector_PinSocket_2.54mm:PinSocket_1x08_P2.54mm_Vertical" (id 2) (at 110.49 48.26 0)
@@
     )
     (path "/3d92ab62-134a-4ba8-bb93-98169739d76f"
-      (reference "J1") (unit 1) (value "GND") (footprint "Connector_PinSocket_2.54mm:PinSocket_1x08_P2.54mm_Vertical")
-    )
-    (path "/c4906877-f34e-41ea-9593-c886178643dc"
-      (reference "J2") (unit 1) (value "VCC") (footprint "Connector_PinSocket_2.54mm:PinSocket_1x08_P2.54mm_Vertical")
+      (reference "GND1") (unit 1) (value "GND") (footprint "Connector_PinSocket_2.54mm:PinSocket_1x08_P2.54mm_Vertical")
     )
     (path "/5a5b773e-8175-42a8-b6b9-e317caca901e"
-      (reference "J3") (unit 1) (value "LOGIC CONN") (footprint "Connector_PinSocket_2.54mm:PinSocket_1x06_P2.54mm_Vertical")
+      (reference "J1") (unit 1) (value "LOGIC CONN") (footprint "Connector_PinSocket_2.54mm:PinSocket_1x06_P2.54mm_Vertical")
     )
     (path "/0661d9e7-9725-45e0-99b3-6e9764bee718"
@@
       (reference "U1") (unit 1) (value "74HC237") (footprint "footprints:NS16")
     )
-  )
+    (path "/c4906877-f34e-41ea-9593-c886178643dc"
+      (reference "VCC1") (unit 1) (value "VCC") (footprint "Connector_PinSocket_2.54mm:PinSocket_1x08_P2.54mm_Vertical")
+    )
+  )

Commit message: finish pcb
Parts:
- removed D1, D2, D3, D5, D6, D7: 2V, Connector_PinSocket_2.54mm:PinSocket_1x02_P2.54mm_Vertical, symbol Device:LED
- removed D4, D8: 3V, Connector_PinSocket_2.54mm:PinSocket_1x02_P2.54mm_Vertical, symbol Device:LED
- added H1, H2, H3: MountingHole, MountingHole:MountingHole_3.2mm_M3, symbol Mechanical:MountingHole
- added J2: 2-3V LEDS, Connector_PinSocket_2.54mm:PinSocket_2x08_P2.54mm_Vertical, symbol Connector_Generic:Conn_02x08_Odd_Even
- R1: footprint Resistor_THT:R_Axial_DIN0204_L3.6mm_D1.6mm_P1.90mm_Vertical -> Resistor_THT:R_Axial_Power_L25.0mm_W9.0mm_P10.16mm_Vertical
Connections:
- net at R1.2: now also J2.1 (Pin_1), J2.11 (Pin_11), J2.13 (Pin_13), J2.15 (Pin_15), J2.3 (Pin_3), J2.5 (Pin_5), J2.7 (Pin_7), J2.9 (Pin_9)
- net at U1.7 (Y7): now also J2.16 (Pin_16)
- net at U1.11 (Y4): now also J2.10 (Pin_10)
- net at U1.10 (Y5): now also J2.12 (Pin_12)
- net at U1.12 (Y3): now also J2.8 (Pin_8)
- net at U1.13 (Y2): now also J2.6 (Pin_6)
- net at U1.14 (Y1): now also J2.4 (Pin_4)
- net at U1.15 (Y0): now also J2.2 (Pin_2)
- net at U1.9 (Y6): now also J2.14 (Pin_14)
